Commit message: modified urdf of 00141 to use my obj exports (my CADs) to debug

File: assets/automate/urdf/00141_plug.urdf (robot description, URDF)
Before this commit: robot 00141_plug, 1 links, 0 joints
Links:
- link 00141_plug: geometry collision mesh filename=../mesh/00141/vd_00141/asset_plug.obj; visual mesh filename=../mesh/00141/vd_00141/asset_plug.obj

File: assets/automate/urdf/00141_socket.urdf (robot description, URDF)
Before this commit: robot 00141_socket, 1 links, 0 joints
Links:
- link 00141_socket: geometry collision mesh filename=../mesh/00141/vd_00141/asset_socket.obj; visual mesh filename=../mesh/00141/vd_00141/asset_socket.obj

Commit message: change: using original parts, still does not work

File: assets/automate/urdf/00141_plug.urdf (robot description, URDF)
Before this commit: robot 00141_plug, 1 links, 0 joints
Links:
- link 00141_plug: geometry collision mesh filename=../mesh/00141/asset_plug.obj; visual mesh filename=../mesh/00141/asset_plug.obj

File: assets/automate/urdf/00141_socket.urdf (robot description, URDF)
Before this commit: robot 00141_socket, 1 links, 0 joints
Links:
- link 00141_socket: geometry collision mesh filename=../mesh/00141/asset_socket.obj; visual mesh filename=../mesh/00141/asset_socket.obj
